File: eagle/arduino_dojo_shield_rev01.brd (EAGLE design)
At the start: 26 parts, among them IC1 74LS595N, J1 ARDUINO_R3_SHIELDNOLABELS, M1 SMALL_SERVO, M2 SMALL_SERVO

Commit message: rev 01 - sem layout
Parts:
- added C3: (no value), SparkFun-Capacitors:CAP-PTH-SMALL-KIT
- added C4: (no value), SparkFun-Capacitors:CPOL-RADIAL-10UF-25V
- added D2: LED-RGB-CC-THRUCLEAR, SparkFun-LED:LED-RGB-THRU
- added D3: (no value), SparkFun-DiscreteSemi:DIODE-1N4148-KIT
- added D4, D5, D6, D7: (no value), SparkFun-LED:LED3MM
- added J3: (no value), SparkFun-Connectors:1X03
- added J4: (no value), SparkFun-Connectors:SCREWTERMINAL-5MM-2
- added M3: SMALL_SERVO, GH_SparkFun-Electromechanical:1X03
- added R14, R15, R16, R17, R18: (no value), SparkFun-Passives:0805
- D1: value LED-RGB-CC-THRUCLEAR -> (none); device SparkFun-LED:LED-RGB-THRU -> SparkFun-LED:LED3MM
- J1: device SparkFun-Boards:UNO_R3_SHIELD_NOLABELS -> GH_SparkFun-Boards:UNO_R3_SHIELD_NOLABELS
- M1, M2: device SparkFun-Electromechanical:1X03 -> GH_SparkFun-Electromechanical:1X03
- R1: device SparkFun-Passives:AXIAL-0.4 -> SparkFun-Passives:0805
- R2: value PHOTOCELLPTH -> (none); device SparkFun-Sensors:PHOTOCELL -> SparkFun-Passives:AXIAL-0.4
- R3: value (none) -> PHOTOCELLPTH; device SparkFun-Passives:0805 -> SparkFun-Sensors:PHOTOCELL
- moved R1 53.9 mm to (8.89, 5.08), flipped to the bottom, turned to 90 degrees
- moved R6 37.2 mm to (22.9, 8.89), turned to 180 degrees
- moved D1 30.6 mm to (6.35, 5.08)
- moved R3 22.5 mm to (39.4, 43.2), flipped to the top, turned to 0 degrees
- moved R7 19.0 mm to (22.5, 31.1), turned to 180 degrees
- moved R12 18.7 mm to (28.4, 45.7)
- moved R10 16.5 mm to (13.2, 45.7)
- moved R8 15.9 mm to (22.5, 29.2), turned to 180 degrees
- moved R9 12.9 mm to (22.6, 27.4)
- moved R5 12.2 mm to (22.9, 14.0)
- moved C1 12.0 mm to (6.35, 14.0), turned to 90 degrees
- moved R2 10.2 mm to (39.4, 50.8)
- moved R4 9.03 mm to (22.9, 19.1)
- moved R11 8.93 mm to (13.2, 48.2)
- moved M1 8.52 mm to (22.9, 59.7)
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Connections:
- removed net N$17 (its old number): J1.D10, M2.1
- removed net N$34: IC1.12, J1.D12
- new net N$16: J1.D12, M2.1
- new net N$2: J1.A3, J3.2
- new net N$24: IC1.14, J1.D11
- new net N$32: J1.D8, M3.1
- new net N$37: J1.A0, S1.1, S1.2
- new net N$38: D1.A, R1.1
- new net N$40: D5.A, R5.2
- new net N$41: D6.A, R6.2
- new net N$42: D4.A, R4.2
- new net N$43: J1.D4, R5.1
- new net N$44: J1.D2, R4.1
- new net N$45: IC1.12, J1.D10
- new net VCC: C1.1, C2.1, IC1.10, IC1.16, J1.5V, J3.3, R1.2, R2.P$2, RV1.3
- net 5V: now also C3.1, C4.1, D3.C, J4.2, M3.2, R18.1; no longer C1.1, C2.1, IC1.10, IC1.16, J1.5V, R1.P$2, RV1.3
- net GND: now also C3.2, C4.2, D1.K, D2.2, D3.A, D4.K, D5.K, D6.K, D7.K, J3.1, J4.1, M3.3, R3.1; no longer D1.2, R2.1
- net N$1: now also J1.A4, R2.P$1, R3.2; no longer J1.A3, R1.P$1, R2.2
- net N$10: now also D2.3, R8.2; no longer D1.3, R4.2
- net N$11: now also D2.4, R9.2; no longer D1.4, R5.2
- net N$12: now also R6.1; no longer S2.1, S2.2
- net N$13: now also IC1.11, J1.D13; no longer J1.D8, S3.1, S3.2
- net N$14: now also R10.1; no longer R6.1
- net N$15: now also R10.2; no longer R6.2
- net N$18: now also R11.1; no longer R7.1
- net N$19: now also R11.2; no longer R7.2
- net N$20: now also R12.1; no longer R8.1
- net N$21: now also R12.2; no longer R8.2
- net N$22: now also R13.1; no longer R9.1
- net N$23: now also R13.2; no longer R9.2
- net N$25: now also R14.2; no longer R10.2
- net N$26: now also R15.1; no longer R11.1
- net N$27: now also R15.2; no longer R11.2
- net N$28: now also R16.1; no longer R12.1
- net N$29: now also R16.2; no longer R12.2
- net N$3: now also R14.1; no longer R10.1
- net N$30: now also R17.1; no longer R13.1
- net N$31: now also R17.2; no longer R13.2
- net N$33: now also D7.A, R18.2; no longer IC1.14, J1.D13
- net N$35: now also J1.A1, S2.1, S2.2; no longer IC1.11, J1.D11
- net N$36: now also J1.A2, S3.1, S3.2; no longer J1.D2, S1.1, S1.2
- net N$4: now also R9.1; no longer R5.1
- net N$5: now also R8.1; no longer R4.1
- net N$8: now also R7.1; no longer R3.1
- net N$9: now also D2.1, R7.2; no longer D1.1, R3.2
Routing:
- added copper zone on layer 16, net N$34
- added copper zone on layer 1, net N$46

Commit message: eagle rev 0
Parts:
- moved R1 1.27 mm to (10.2, 5.08)
Changed lines of the file:
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@@
 <element name="J3" library="SparkFun-Connectors" package="1X03" value="" x="50.8" y="59.69" rot="R90"/>
 <element name="R18" library="SparkFun-Passives" package="0805" value="" x="8.89" y="53.34" rot="MR270"/>
-<element name="R1" library="SparkFun-Passives" package="0805" value="" x="8.89" y="5.08" rot="MR90"/>
+<element name="R1" library="SparkFun-Passives" package="0805" value="" x="10.16" y="5.08" rot="MR90"/>
 <element name="D4" library="SparkFun-LED" package="LED3MM" value="" x="27.94" y="19.05">
 <attribute name="PROD_ID" value="DIO-08794" x="27.94" y="19.05" size="1.778" layer="27" display="off"/>
@@
 <wire x1="6.35" y1="12.573" x2="10.16" y2="25.4" width="0" layer="19" extent="1-1"/>
 <wire x1="10.16" y1="10.16" x2="6.35" y2="12.573" width="0" layer="19" extent="1-1"/>
-<wire x1="8.89" y1="5.98" x2="10.16" y2="10.16" width="0" layer="19" extent="16-16"/>
+<wire x1="10.16" y1="5.98" x2="10.16" y2="10.16" width="0" layer="19" extent="16-16"/>
 </signal>
 <signal name="N$33">
@@
 <contactref element="D1" pad="A"/>
 <contactref element="R1" pad="1"/>
-<wire x1="6.35" y1="3.81" x2="8.89" y2="4.18" width="0" layer="19" extent="16-16"/>
+<wire x1="6.35" y1="3.81" x2="10.16" y2="4.18" width="0" layer="19" extent="16-16"/>
 </signal>
 <signal name="N$2">
